Commit message: updated git modules

File: xarm_ros2/xarm_description/urdf/lite6/lite6.gazebo.xacro (robot description, xacro)
@@ -23,4 +23,7 @@
       <selfCollide>true</selfCollide>
     </gazebo>
+    <gazebo reference="camera_depth_optical_frame">
+      <selfCollide>false</selfCollide>
+    </gazebo>
   </xacro:macro>
 </robot>

File: xarm_ros2/xarm_description/urdf/lite6/lite6.urdf.xacro (robot description, xacro)
@@ -9,5 +9,6 @@
     joint6_lower_limit:=${-2.0*pi}  joint6_upper_limit:=${2.0*pi}
     model_num:=0
-    inertial_params_filename:='' kinematics_params_filename:='' "
+    inertial_params_filename:='' kinematics_params_filename:=''
+    simulated:='false' "
     >
     <!-- load params and define property -->
@@ -208,33 +209,36 @@
       <dynamics damping="1.0" friction="1.0"/>
     </joint>
-    <link name="camera_depth_optical_frame">
-      <inertial>
-        <origin xyz="0 0 0" rpy="0 0 0" />
-        <mass value="0.01" />
-        <inertia
-          ixx="0" ixy="0" ixz="0"
-          iyy="0" iyz="0" izz="0" />
-      </inertial>
-      <visual>
-        <origin xyz="0 0 0" rpy="0 0 0" />
-        <geometry>
-          <box size="0.03 0.01 0.01" />
-        </geometry>
-        <material name="camera_depth_optical_frame_color">
-          <color rgba="0.0 0.0 1.0 1.0" />
-        </material>
-      </visual>
-      <collision>
-        <origin xyz="0 0 0" rpy="0 0 0" />
-        <geometry>
-          <box size="0.01 0.01 0.01" />
-        </geometry>
-      </collision>
-    </link>
-    <joint name="joint_link6_camera_link" type="fixed">
-      <origin xyz="-0.06 0.01 0.01" rpy="0 0 4.71" />
-      <parent link="${prefix}link6" />
-      <child link="camera_depth_optical_frame" />
-    </joint>
+    <!-- * Remove to uncomment before running on the actual arm -->
+    <!-- <xacro:unless value="${simulated}">
+      <link name="camera_depth_optical_frame">
+        <inertial>
+          <origin xyz="0 0 0" rpy="0 0 0" />
+          <mass value="0.01" />
+          <inertia
+            ixx="0" ixy="0" ixz="0"
+            iyy="0" iyz="0" izz="0" />
+        </inertial>
+        <visual>
+          <origin xyz="0 0 0" rpy="0 0 0" />
+          <geometry>
+            <box size="0.03 0.01 0.01" />
+          </geometry>
+          <material name="camera_depth_optical_frame_color">
+            <color rgba="0.0 0.0 1.0 1.0" />
+          </material>
+        </visual>
+        <collision>
+          <origin xyz="0 0 0" rpy="0 0 0" />
+          <geometry>
+            <box size="0.01 0.01 0.01" />
+          </geometry>
+        </collision>
+      </link>
+      <joint name="joint_link6_camera_link" type="fixed">
+        <origin xyz="-0.06 0.01 0.01" rpy="0 0 4.71" />
+        <parent link="${prefix}link6" />
+        <child link="camera_depth_optical_frame" />
+      </joint>
+    </xacro:unless> -->
     <!-- <link name="${prefix}link_eef" />
     <joint name="${prefix}joint_eef" type="fixed">

File: xarm_ros2/xarm_description/urdf/lite6/lite6_robot_macro.xacro (robot description, xacro)
@@ -15,5 +15,7 @@
     inertial_params_filename:=''
     kinematics_params_filename:=''
-    hard_interface:='PositionJointInterface' "
+    hard_interface:='PositionJointInterface'
+    simulated:='false'
+    "
     >
     <!-- include lite6 relative macros: -->
@@ -49,4 +51,5 @@
         inertial_params_filename="${inertial_params_filename}"
         kinematics_params_filename="${kinematics_params_filename}"
+        simulated="${simulated}"
         />
     </xacro:if>

File: xarm_ros2/xarm_description/urdf/xarm_device.urdf.xacro (robot description, xacro)
@@ -38,4 +38,6 @@
   <xacro:arg name="attach_rpy" default="0 0 0"/>
   <xacro:arg name="mesh_suffix" default="stl"/>
+  <!-- ! Added by Tanay -->
+  <xacro:arg name="simulated" default="false"/>
   <xacro:arg name="kinematics_suffix" default=""/>
   <!-- load xarm device -->
@@ -59,4 +61,4 @@
     baud_checkset="$(arg baud_checkset)" default_gripper_baud="$(arg default_gripper_baud)"
     model1300="$(arg model1300)" attach_to="$(arg attach_to)" attach_xyz="$(arg attach_xyz)" attach_rpy="$(arg attach_rpy)"
-    robot_sn="$(arg robot_sn)" use_gazebo_camera="$(arg use_gazebo_camera)" mesh_suffix="$(arg mesh_suffix)" kinematics_suffix="$(arg kinematics_suffix)" />
+    robot_sn="$(arg robot_sn)" use_gazebo_camera="$(arg use_gazebo_camera)" mesh_suffix="$(arg mesh_suffix)" kinematics_suffix="$(arg kinematics_suffix)" simulated="$(arg simulated)" />
 </robot>

File: xarm_ros2/xarm_description/urdf/xarm_device_macro.xacro (robot description, xacro)
@@ -42,4 +42,5 @@
     mesh_suffix:='stl'
     kinematics_suffix:=''
+    simulated:='false'
     "
     >
@@ -145,5 +146,6 @@
           inertial_params_filename="${inertial_params_filename}"
           kinematics_params_filename="${kinematics_params_filename}"
-          hard_interface="${hard_interface}" />
+          hard_interface="${hard_interface}"
+          simulated="${simulated}"/>
       </xacro:if>
       <xacro:unless value="${robot_type == 'lite' or robot_type == 'uf850'}">
