Commit message: modiified descriptions, added realsense support, made transformations

File: xarm_ros2/xarm_description/urdf/lite6/lite6.urdf.xacro (robot description, xacro)
@@ -210,5 +210,5 @@
     <link name="camera_depth_optical_frame">
       <inertial>
-        <origin xyz="0 0 0" rpy="0 0 3.14" />
+        <origin xyz="0 0 0" rpy="0 0 0" />
         <mass value="0.01" />
         <inertia
@@ -233,5 +233,5 @@
     </link>
     <joint name="joint_link6_camera_link" type="fixed">
-      <origin xyz="0 0 0.01" rpy="0 0 0" />
+      <origin xyz="0 0 0.01" rpy="0 0 4.71" />
       <parent link="${prefix}link6" />
       <child link="camera_depth_optical_frame" />

Commit message: added mapping from camera to realsense

File: xarm_ros2/xarm_description/urdf/lite6/lite6.urdf.xacro (robot description, xacro)
@@ -219,5 +219,5 @@
         <origin xyz="0 0 0" rpy="0 0 0" />
         <geometry>
-          <box size="0.01 0.01 0.01" />
+          <box size="0.03 0.01 0.01" />
         </geometry>
         <material name="camera_depth_optical_frame_color">
@@ -233,5 +233,5 @@
     </link>
     <joint name="joint_link6_camera_link" type="fixed">
-      <origin xyz="0 0 0.01" rpy="0 0 4.71" />
+      <origin xyz="-0.06 0.01 0.01" rpy="0 0 4.71" />
       <parent link="${prefix}link6" />
       <child link="camera_depth_optical_frame" />

Commit message: added manav's gripper meshes

File: xarm_ros2/xarm_description/urdf/lite6/lite6.urdf.xacro (robot description, xacro)
@@ -208,4 +208,6 @@
       <dynamics damping="1.0" friction="1.0"/>
     </joint>
+    <!-- <xacro:include filename="$(find crackle_description)/urdf/crackle_gripper.urdf.xacro" /> -->
+    <!-- <xacro:three_claw_gripper arm_link="${prefix}link6" /> -->
     <!-- <link name="${prefix}link_eef" />
     <joint name="${prefix}joint_eef" type="fixed">

File: xarm_ros2/xarm_moveit_config/srdf/_lite6_macro.srdf.xacro (robot description, xacro)
@@ -37,8 +37,8 @@
     <group_state name="home" group="${prefix}lite6">
       <joint name="${prefix}joint1" value="0" />
-      <joint name="${prefix}joint2" value="0" />
-      <joint name="${prefix}joint3" value="0" />
+      <joint name="${prefix}joint2" value="-0.0349066" />
+      <joint name="${prefix}joint3" value="0.331613" />
       <joint name="${prefix}joint4" value="0" />
-      <joint name="${prefix}joint5" value="0" />
+      <joint name="${prefix}joint5" value="0.366519" />
       <joint name="${prefix}joint6" value="0" />
     </group_state>

Commit message: converted mtc to dir and fixed submodules

File: xarm_ros2/xarm_description/urdf/lite6/lite6.urdf.xacro (robot description, xacro)
@@ -210,10 +210,10 @@
     <xacro:include filename="$(find crackle_description)/urdf/crackle_gripper.urdf.xacro" />
     <xacro:three_claw_gripper arm_link="${prefix}link6" />
-    <!-- <link name="${prefix}link_eef" />
+    <link name="${prefix}link_eef" />
     <joint name="${prefix}joint_eef" type="fixed">
       <origin xyz="0 0 0" rpy="0 0 0" />
       <parent link="${prefix}link6" />
       <child link="${prefix}link_eef" />
-    </joint> -->
+    </joint>
   </xacro:macro>
 </robot>
