Commit message: added moveit scene updater

File: crackle_description/urdf/crackle_gripper.urdf.xacro (robot description, xacro)
@@ -17,16 +17,16 @@
         </geometry>
       </visual>
-      <collision>
-        <origin xyz="0 0 0" rpy="0 0 0"/>
-        <geometry>
-          <mesh filename="${pkg_path}/${base_mesh}" scale="${mesh_scale}"/>
-        </geometry>
-      </collision>
+      <!-- <collision> -->
+        <!-- <origin xyz="0 0 0" rpy="0 0 0"/> -->
+        <!-- <geometry> -->
+          <!-- <mesh filename="${pkg_path}/${base_mesh}" scale="${mesh_scale}"/> -->
+        <!-- </geometry> -->
+      <!-- </collision> -->
       <inertial>
         <origin xyz="0 0 0" rpy="0 0 0"/>
         <mass value="0.2"/>
-        <inertia ixx="0.001" ixy="0.0" ixz="0.0"
-                 iyy="0.001" iyz="0.0"
-                 izz="0.001"/>
+        <inertia ixx="220.703" ixy="66.047" ixz="-11.782"
+                 iyy="300.204" iyz="-23.973"
+                 izz="394.277"/>
       </inertial>
       <color rgba="0.0 0.0 0.5 1"/>
@@ -48,10 +48,10 @@
         </geometry>
       </visual>
-      <collision>
+      <!-- <collision>
         <origin xyz="0 0 0" rpy="0 0 0"/>
         <geometry>
           <mesh filename="${pkg_path}/${claw_mesh}" scale="${mesh_scale}"/>
         </geometry>
-      </collision>
+      </collision> -->
       <inertial>
         <origin xyz="0 0 0" rpy="0 0 0"/>
@@ -79,4 +79,40 @@
     <parent link="${arm_last_link}"/>
     <child link="gripper_base"/>
+    <origin xyz="0 0 0.005" rpy="0.0 0 0.78"/>
+  </joint>
+  <link name="camera_depth_optical_frame">
+    <visual>
+      <origin xyz="0 0 0" rpy="0 0 0"/>
+      <geometry>
+        <mesh filename="${pkg_path}/realsense_d435i.stl" scale="${mesh_scale}"/>
+      </geometry>
+      <material name="blue">
+        <color rgba="0.0 0.0 0.5 1"/>
+      </material>
+    </visual>
+    <inertial>
+      <origin xyz="0 0 0" rpy="0 0 0"/>
+      <mass value="0.1"/>
+      <inertia ixx="0.001" ixy="0.0" ixz="0.0"
+               iyy="0.001" iyz="0.0"
+               izz="0.001"/>
+    </inertial>
+  </link>
+  <joint name="camera_depth_optical_frame_joint" type="fixed">
+    <parent link="gripper_base"/>
+    <child link="camera_depth_optical_frame"/>
+    <origin xyz="-0.08 0 0.03" rpy="0 0 -1.57"/>
+  </joint>
+  <link name="leapmotion_link">
+    <!-- <visual>
+      <origin xyz="0 0 0" rpy="0 0 0"/>
+      <geometry>
+        <box size="0.1 0.1 0.1"/>
+      </geometry>
+    </visual> -->
+  </link>
+  <joint name="leapmotion_link_joint" type="fixed">
+    <parent link="gripper_base"/>
+    <child link="leapmotion_link"/>
     <origin xyz="0 0 0" rpy="0 0 0"/>
   </joint>
@@ -85,18 +121,18 @@
     claw_name="claw_1"
     claw_mesh="ClawArm.stl"
-    pivot_xyz="0 -0.05 0.05"
-    pivot_rpy="0 1.57 0"
+    pivot_xyz="0 -0.035 0.04"
+    pivot_rpy="0 1.0 0.34"
     pivot_axis="0 1 0"/>
-  <xacro:claw_macro
+   <xacro:claw_macro
     claw_name="claw_2"
     claw_mesh="ClawArm.stl"
-    pivot_xyz="0.05 -0.05 0"
-    pivot_rpy="0 1.57 1.57"
+    pivot_xyz="0.03 0.01 0.04"
+    pivot_rpy="0 1.57 2.34"
     pivot_axis="0 1 0"/>
   <xacro:claw_macro
     claw_name="claw_3"
     claw_mesh="ClawArm.stl"
-    pivot_xyz="0 0.05 0"
-    pivot_rpy="1.57 1.57 1.57"
+    pivot_xyz="-0.03 0.01 0.04"
+    pivot_rpy="0 1.0 -1.57"
     pivot_axis="0 1 0"/> -->
   </xacro:macro>

File: xarm_ros2/xarm_description/urdf/lite6/lite6.urdf.xacro (robot description, xacro)
@@ -208,6 +208,6 @@
       <dynamics damping="1.0" friction="1.0"/>
     </joint>
-    <!-- <xacro:include filename="$(find crackle_description)/urdf/crackle_gripper.urdf.xacro" /> -->
-    <!-- <xacro:three_claw_gripper arm_link="${prefix}link6" /> -->
+    <xacro:include filename="$(find crackle_description)/urdf/crackle_gripper.urdf.xacro" />
+    <xacro:three_claw_gripper arm_link="${prefix}link6" />
     <!-- <link name="${prefix}link_eef" />
     <joint name="${prefix}joint_eef" type="fixed">

Commit message: moveit works, face an, gripper, and audio localization merged in

File: crackle_description/urdf/crackle_gripper.urdf.xacro (robot description, xacro)
@@ -9,5 +9,5 @@
        Macro: Gripper Base Link
        ========================= -->
-  <xacro:macro name="gripper_base_macro" params="link_name base_mesh:='ClawBase.stl'">
+  <xacro:macro name="gripper_base_macro" params="link_name base_mesh:='damn.stl'">
     <link name="${link_name}">
       <visual>
@@ -120,20 +120,20 @@
   <!-- <xacro:claw_macro
     claw_name="claw_1"
-    claw_mesh="ClawArm.stl"
-    pivot_xyz="0 -0.035 0.04"
-    pivot_rpy="0 1.0 0.34"
-    pivot_axis="0 1 0"/>
-   <xacro:claw_macro
+    claw_mesh="elArmo.stl"
+    pivot_xyz=".002 .025 0.009"
+    pivot_rpy="1.0 2.0 2.0"
+    pivot_axis="0 1 0"/> -->
+   <!-- <xacro:claw_macro
     claw_name="claw_2"
-    claw_mesh="ClawArm.stl"
-    pivot_xyz="0.03 0.01 0.04"
+    claw_mesh="elArmo.stl"
+    pivot_xyz="-.025 0.019 0.013"
     pivot_rpy="0 1.57 2.34"
     pivot_axis="0 1 0"/>
   <xacro:claw_macro
     claw_name="claw_3"
-    claw_mesh="ClawArm.stl"
-    pivot_xyz="-0.03 0.01 0.04"
+    claw_mesh="elArmo.stl"
+    pivot_xyz=".025 0.015 0.013"
     pivot_rpy="0 1.0 -1.57"
-    pivot_axis="0 1 0"/> -->
+    pivot_axis="0 1 0"/>  -->
   </xacro:macro>
 </robot>

Commit message: Add MoveIt! manipulation functionalities for Crackle robot
- Implemented moveit_manipulation.hpp and moveit_manipulation.cpp files.
- Added initialization function for MoveGroupInterface.
- Created move_to_pose function to plan and execute motions to a target pose.
- Defined a main function to run the manipulation node and move the robot's end effector to a hardcoded target pose.
- Included necessary headers and set up logging for planning outcomes.

File: crackle_description/urdf/crackle_gripper.urdf.xacro (robot description, xacro)
@@ -9,5 +9,5 @@
        Macro: Gripper Base Link
        ========================= -->
-  <xacro:macro name="gripper_base_macro" params="link_name base_mesh:='damn.stl'">
+  <xacro:macro name="gripper_base_macro" params="link_name base_mesh:='ClawBase.stl'">
     <link name="${link_name}">
       <visual>
@@ -32,41 +32,4 @@
       <color rgba="0.0 0.0 0.5 1"/>
     </link>
-  </xacro:macro>
-  <!-- =========================
-       Macro: Claw Link + Joint
-       =========================
-       params:
-         claw_name, claw_mesh
-         pivot_xyz, pivot_rpy, pivot_axis
-  -->
-  <xacro:macro name="claw_macro" params="claw_name claw_mesh pivot_xyz:='0 0 0' pivot_rpy:='0 0 0' pivot_axis:='0 0 1'">
-    <link name="${claw_name}">
-      <visual>
-        <origin xyz="0 0 0" rpy="0 0 0"/>
-        <geometry>
-          <mesh filename="${pkg_path}/${claw_mesh}" scale="${mesh_scale}"/>
-        </geometry>
-      </visual>
-      <!-- <collision>
-        <origin xyz="0 0 0" rpy="0 0 0"/>
-        <geometry>
-          <mesh filename="${pkg_path}/${claw_mesh}" scale="${mesh_scale}"/>
-        </geometry>
-      </collision> -->
-      <inertial>
-        <origin xyz="0 0 0" rpy="0 0 0"/>
-        <mass value="0.05"/>
-        <inertia ixx="0.0001" ixy="0.0" ixz="0.0"
-                 iyy="0.0001" iyz="0.0"
-                 izz="0.0001"/>
-      </inertial>
-    </link>
-    <joint name="${claw_name}_joint" type="revolute">
-      <parent link="gripper_base"/>
-      <child link="${claw_name}"/>
-      <origin xyz="${pivot_xyz}" rpy="${pivot_rpy}"/>
-      <axis xyz="${pivot_axis}"/>
-      <limit effort="1.0" velocity="1.0" lower="0" upper="1.57"/>
-    </joint>
   </xacro:macro>
   <!-- =========================
@@ -104,36 +67,4 @@
     <origin xyz="-0.08 0 0.03" rpy="0 0 -1.57"/>
   </joint>
-  <link name="leapmotion_link">
-    <!-- <visual>
-      <origin xyz="0 0 0" rpy="0 0 0"/>
-      <geometry>
-        <box size="0.1 0.1 0.1"/>
-      </geometry>
-    </visual> -->
-  </link>
-  <joint name="leapmotion_link_joint" type="fixed">
-    <parent link="gripper_base"/>
-    <child link="leapmotion_link"/>
-    <origin xyz="0 0 0" rpy="0 0 0"/>
-  </joint>
-  <!-- 3) Three claws, each with a revolute joint -->
-  <!-- <xacro:claw_macro
-    claw_name="claw_1"
-    claw_mesh="elArmo.stl"
-    pivot_xyz=".002 .025 0.009"
-    pivot_rpy="1.0 2.0 2.0"
-    pivot_axis="0 1 0"/> -->
-   <!-- <xacro:claw_macro
-    claw_name="claw_2"
-    claw_mesh="elArmo.stl"
-    pivot_xyz="-.025 0.019 0.013"
-    pivot_rpy="0 1.57 2.34"
-    pivot_axis="0 1 0"/>
-  <xacro:claw_macro
-    claw_name="claw_3"
-    claw_mesh="elArmo.stl"
-    pivot_xyz=".025 0.015 0.013"
-    pivot_rpy="0 1.0 -1.57"
-    pivot_axis="0 1 0"/>  -->
   </xacro:macro>
 </robot>

Commit message: added launch file and bash script

File: crackle_description/urdf/crackle_gripper.urdf.xacro (robot description, xacro)
@@ -42,5 +42,5 @@
     <parent link="${arm_last_link}"/>
     <child link="gripper_base"/>
-    <origin xyz="0 0 0.005" rpy="0.0 0 0.78"/>
+    <origin xyz="0 0 0.025" rpy="0.0 0 -0.78"/> <!-- 0.78 -->
   </joint>
   <link name="camera_depth_optical_frame">

Commit message: old gpt generate code

File: crackle_description/urdf/crackle_gripper.urdf.xacro (robot description, xacro)
@@ -12,5 +12,5 @@
     <link name="${link_name}">
       <visual>
-        <origin xyz="0 0 0" rpy="0 0 0"/>
+        <origin xyz="0 0 0" rpy="1.57 0 0"/>
         <geometry>
           <mesh filename="${pkg_path}/${base_mesh}" scale="${mesh_scale}"/>

Commit message: added code generation

File: crackle_description/urdf/crackle_gripper.urdf.xacro (robot description, xacro)
@@ -12,5 +12,5 @@
     <link name="${link_name}">
       <visual>
-        <origin xyz="0 0 0" rpy="1.57 0 0"/>
+        <origin xyz="0 0 0" rpy="0 0 0"/>
         <geometry>
           <mesh filename="${pkg_path}/${base_mesh}" scale="${mesh_scale}"/>

Commit message: added new gripper stl

File: crackle_description/urdf/crackle_gripper.urdf.xacro (robot description, xacro)
@@ -9,5 +9,5 @@
        Macro: Gripper Base Link
        ========================= -->
-  <xacro:macro name="gripper_base_macro" params="link_name base_mesh:='ClawBase.stl'">
+  <xacro:macro name="gripper_base_macro" params="link_name base_mesh:='crackle_gripper.stl'">
     <link name="${link_name}">
       <visual>

Commit message: added corrected xacro

File: crackle_description/urdf/crackle_gripper.urdf.xacro (robot description, xacro)
@@ -12,5 +12,5 @@
     <link name="${link_name}">
       <visual>
-        <origin xyz="0 0 0" rpy="0 0 0"/>
+        <origin xyz="0 0 0" rpy="0 0 1.80"/>
         <geometry>
           <mesh filename="${pkg_path}/${base_mesh}" scale="${mesh_scale}"/>

Commit message: updated?

File: crackle_description/urdf/crackle_gripper.urdf.xacro (robot description, xacro)
@@ -9,5 +9,5 @@
        Macro: Gripper Base Link
        ========================= -->
-  <xacro:macro name="gripper_base_macro" params="link_name base_mesh:='crackle_gripper.stl'">
+  <xacro:macro name="gripper_base_macro" params="link_name base_mesh:='Claw_Casing.stl'">
     <link name="${link_name}">
       <visual>
@@ -17,19 +17,38 @@
         </geometry>
       </visual>
-      <!-- <collision> -->
-        <!-- <origin xyz="0 0 0" rpy="0 0 0"/> -->
-        <!-- <geometry> -->
-          <!-- <mesh filename="${pkg_path}/${base_mesh}" scale="${mesh_scale}"/> -->
-        <!-- </geometry> -->
-      <!-- </collision> -->
-      <inertial>
-        <origin xyz="0 0 0" rpy="0 0 0"/>
-        <mass value="0.2"/>
-        <inertia ixx="220.703" ixy="66.047" ixz="-11.782"
-                 iyy="300.204" iyz="-23.973"
-                 izz="394.277"/>
-      </inertial>
       <color rgba="0.0 0.0 0.5 1"/>
     </link>
+    <link name="spur_gear_left">
+      <visual>
+        <origin xyz="0 0 0" rpy="0 0 1.80"/>
+        <geometry>
+          <mesh filename="${pkg_path}/SpurGear_Left.stl" scale="${mesh_scale}"/>
+        </geometry>
+      </visual>
+      <color rgba="0.0 0.0 0.5 1"/>
+    </link>
+  <link name="spur_gear_right">
+      <visual>
+        <origin xyz="0 0 0" rpy="0 0 1.80"/>
+        <geometry>
+          <mesh filename="${pkg_path}/SpurGear_Right.stl" scale="${mesh_scale}"/>
+        </geometry>
+      </visual>
+      <color rgba="0.0 0.0 0.5 1"/>
+    </link>
+    <joint name="spur_gear_left_joint" type="revolute">
+      <parent link="${link_name}"/>
+      <child link="spur_gear_left"/>
+      <origin xyz="0 0 0" rpy="0 0 0"/>
+      <axis xyz="0 0 1"/>
+      <limit lower="-3.14159" upper="3.14159" effort="5.0" velocity="5.0"/>
+    </joint>
+    <joint name="spur_gear_right_joint" type="revolute">
+      <parent link="${link_name}"/>
+      <child link="spur_gear_right"/>
+      <origin xyz="0 0 0" rpy="0 0 0"/>
+      <axis xyz="0 0 1"/>
+      <limit lower="-3.14159" upper="3.14159" effort="5.0" velocity="5.0"/>
+    </joint>
   </xacro:macro>
   <!-- =========================
