Commit message: Integrate CRACKLE_CLAW firmware and update claw degree publisher
- Added CRACKLE_CLAW submodule for claw control
- Implemented claw control logic in claw_degree_publisher
- Enhanced URDF with new gripper mesh and joint definitions
- Updated package dependencies for ROS integration

File: crackle_description/urdf/crackle_gripper.urdf.xacro (robot description, xacro)
@@ -5,51 +5,72 @@
   <xacro:property name="pkg_path" value="package://crackle_description/meshes"/>
   <xacro:property name="mesh_scale" value="1 1 1"/>
+  <!-- The lateral_rack_pinion_gripper mesh is authored in millimetres; scale to metres. -->
+  <xacro:property name="mm_scale" value="0.001 0.001 0.001"/>
   <xacro:property name="arm_last_link" value="${arm_link}"/>
+  <!-- Placement of the gripper mesh within the gripper_base link.
+       Tune these in RViz if the body is not oriented as expected. -->
+  <xacro:property name="gripper_mesh_xyz" value="0 0 0"/>
+  <xacro:property name="gripper_mesh_rpy" value="0 0 0"/>
+  <!-- Lateral rack (jaw) travel, in metres, from fully open (0) to fully closed. -->
+  <xacro:property name="rack_travel" value="0.03"/>
+  <!-- Where the jaws sit relative to the base origin (long axis of the mesh). -->
+  <xacro:property name="jaw_z" value="-0.15"/>
+  <xacro:property name="jaw_open_y" value="0.05"/>
   <!-- =========================
        Macro: Gripper Base Link
        ========================= -->
-  <xacro:macro name="gripper_base_macro" params="link_name base_mesh:='ClawBase.stl'">
+  <xacro:macro name="gripper_base_macro" params="link_name base_mesh:='lateral_rack_pinion_gripper.stl'">
     <link name="${link_name}">
       <visual>
-        <origin xyz="0 0 0" rpy="0 0 1.80"/>
+        <origin xyz="${gripper_mesh_xyz}" rpy="${gripper_mesh_rpy}"/>
         <geometry>
-          <mesh filename="${pkg_path}/${base_mesh}" scale="${mesh_scale}"/>
+          <mesh filename="${pkg_path}/${base_mesh}" scale="${mm_scale}"/>
         </geometry>
+        <material name="gripper_blue">
+          <color rgba="0.0 0.0 0.5 1"/>
+        </material>
       </visual>
-      <color rgba="0.0 0.0 0.5 1"/>
     </link>
-<!--
-    <link name="spur_gear_left">
+    <!-- ===== Left rack (jaw) ===== -->
+    <link name="left_rack">
       <visual>
-        <origin xyz="0 0 0" rpy="0 0 1.80"/>
+        <origin xyz="0 0 0" rpy="0 0 0"/>
         <geometry>
-          <mesh filename="${pkg_path}/SpurGear.stl" scale="${mesh_scale}"/>
+          <box size="0.02 0.01 0.04"/>
         </geometry>
+        <material name="rack_grey">
+          <color rgba="0.3 0.3 0.3 1"/>
+        </material>
       </visual>
-      <color rgba="0.0 0.0 0.5 1"/>
     </link>
-  <link name="spur_gear_right">
+    <!-- ===== Right rack (jaw) ===== -->
+    <link name="right_rack">
       <visual>
-        <origin xyz="0 0 0" rpy="0 0 1.80"/>
+        <origin xyz="0 0 0" rpy="0 0 0"/>
         <geometry>
-          <mesh filename="${pkg_path}/SpurGear.stl" scale="${mesh_scale}"/>
+          <box size="0.02 0.01 0.04"/>
         </geometry>
+        <material name="rack_grey">
+          <color rgba="0.3 0.3 0.3 1"/>
+        </material>
       </visual>
-      <color rgba="0.0 0.0 0.5 1"/>
-  </link>
-    <joint name="spur_gear_left_joint" type="revolute">
+    </link>
+    <!-- Prismatic rack joints. Both racks are driven symmetrically by the two
+         pinion servos, so a single (positive) joint value closes both jaws.
+         Positive axis direction points inward (toward the centreline). -->
+    <joint name="left_rack_joint" type="prismatic">
       <parent link="${link_name}"/>
-      <child link="spur_gear_left"/>
-      <origin xyz="0.0 0.02 0.03" rpy="3.14 1.57 0.3"/>
-      <axis xyz="0 0 1"/>
-      <limit lower="-3.14159" upper="3.14159" effort="5.0" velocity="5.0"/>
+      <child link="left_rack"/>
+      <origin xyz="0 ${jaw_open_y} ${jaw_z}" rpy="0 0 0"/>
+      <axis xyz="0 -1 0"/>
+      <limit lower="0.0" upper="${rack_travel}" effort="10.0" velocity="0.1"/>
     </joint>
-    <joint name="spur_gear_right_joint" type="revolute">
+    <joint name="right_rack_joint" type="prismatic">
       <parent link="${link_name}"/>
-      <child link="spur_gear_right"/>
-      <origin xyz="0.0 -0.02 0.03" rpy="0 1.57 0.3"/>
-      <axis xyz="0 0 1"/>
-      <limit lower="-3.14159" upper="3.14159" effort="5.0" velocity="5.0"/>
-    </joint>  -->
+      <child link="right_rack"/>
+      <origin xyz="0 ${-jaw_open_y} ${jaw_z}" rpy="0 0 0"/>
+      <axis xyz="0 1 0"/>
+      <limit lower="0.0" upper="${rack_travel}" effort="10.0" velocity="0.1"/>
+    </joint>
   </xacro:macro>
   <!-- =========================

Commit message: Added new gripper and edited description

File: crackle_description/urdf/crackle_gripper.urdf.xacro (robot description, xacro)
@@ -9,11 +9,17 @@
   <xacro:property name="arm_last_link" value="${arm_link}"/>
   <!-- Placement of the gripper mesh within the gripper_base link.
-       Tune these in RViz if the body is not oriented as expected. -->
-  <xacro:property name="gripper_mesh_xyz" value="0 0 0"/>
-  <xacro:property name="gripper_mesh_rpy" value="0 0 0"/>
+       In the raw mesh the rack/pinion mechanism sits at one end (mesh Z=-196mm)
+       and the two fingers at the other (mesh Z=+38mm), with the lateral rack
+       running along mesh X. This transform mounts the mechanism end on the
+       flange (link origin) and points the fingers out along +Z (the arm's
+       approach direction), with the rack opening along Y. The 90° yaw turns
+       the rack from mesh X onto Y. -->
+  <xacro:property name="gripper_mesh_xyz" value="-0.002 0.020 0.196"/>
+  <xacro:property name="gripper_mesh_rpy" value="0 0 1.5708"/>
   <!-- Lateral rack (jaw) travel, in metres, from fully open (0) to fully closed. -->
-  <xacro:property name="rack_travel" value="0.03"/>
-  <!-- Where the jaws sit relative to the base origin (long axis of the mesh). -->
-  <xacro:property name="jaw_z" value="-0.15"/>
+  <xacro:property name="rack_travel" value="0.04"/>
+  <!-- Where the jaws sit relative to the base origin: near the finger tips
+       (+Z) and offset laterally along Y. -->
+  <xacro:property name="jaw_z" value="0.19"/>
   <xacro:property name="jaw_open_y" value="0.05"/>
   <!-- =========================
@@ -56,20 +62,25 @@
       </visual>
     </link>
-    <!-- Prismatic rack joints. Both racks are driven symmetrically by the two
-         pinion servos, so a single (positive) joint value closes both jaws.
-         Positive axis direction points inward (toward the centreline). -->
-    <joint name="left_rack_joint" type="prismatic">
+    <!-- Rack (jaw) joints, pinned FIXED at the open position for now.
+         They were prismatic (rack opens along Y, driven symmetrically by the
+         two pinion servos), but a movable joint has no transform until its
+         position is published on /joint_states — which only happens when the
+         claw node is running and the ESP32 is streaming. That broke TF
+         (no transform to left_rack) and MoveIt's current-state monitor
+         (incomplete state -> planning failures) whenever the gripper wasn't
+         actively driven. Fixed joints always resolve and add no DOF to MoveIt.
+         To re-enable articulation: set type="prismatic", restore the <axis>
+         (0 -1 0 / 0 1 0) and <limit lower="0.0" upper="${rack_travel}" ...>,
+         and make claw_degree_publisher publish these joints on /joint_states
+         continuously (see publish_joint_states param). -->
+    <joint name="left_rack_joint" type="fixed">
       <parent link="${link_name}"/>
       <child link="left_rack"/>
       <origin xyz="0 ${jaw_open_y} ${jaw_z}" rpy="0 0 0"/>
-      <axis xyz="0 -1 0"/>
-      <limit lower="0.0" upper="${rack_travel}" effort="10.0" velocity="0.1"/>
     </joint>
-    <joint name="right_rack_joint" type="prismatic">
+    <joint name="right_rack_joint" type="fixed">
       <parent link="${link_name}"/>
       <child link="right_rack"/>
       <origin xyz="0 ${-jaw_open_y} ${jaw_z}" rpy="0 0 0"/>
-      <axis xyz="0 1 0"/>
-      <limit lower="0.0" upper="${rack_travel}" effort="10.0" velocity="0.1"/>
     </joint>
   </xacro:macro>
@@ -79,9 +90,12 @@
   <!-- 1) Base link -->
   <xacro:gripper_base_macro link_name="gripper_base"/>
-  <!-- 2) Fixed joint to arm -->
+  <!-- 2) Fixed joint to arm. The mesh transform above already puts the mount
+       face at the gripper_base origin with the fingers along +Z, so the
+       gripper mounts flush on the flange. Adjust the yaw here to clock the
+       gripper about the tool axis if the jaw-opening direction needs rotating. -->
   <joint name="gripper_base_joint" type="fixed">
     <parent link="${arm_last_link}"/>
     <child link="gripper_base"/>
-    <origin xyz="0 0 0.025" rpy="0.0 0 -0.78"/> <!-- 0.78 -->
+    <origin xyz="0.0 0.0 0.0" rpy="0 0 0"/>
   </joint>
   <link name="camera_depth_optical_frame">
@@ -92,5 +106,5 @@
       </geometry>
       <material name="blue">
-        <color rgba="0.0 0.0 0.5 1"/>
+        <color rgba="0.5 0.0 0.0 1"/>
       </material>
     </visual>
@@ -106,5 +120,5 @@
     <parent link="gripper_base"/>
     <child link="camera_depth_optical_frame"/>
-    <origin xyz="-0.08 0 0.03" rpy="0 0 -1.57"/>
+    <origin xyz="0.02 0.02 0.05" rpy="0.04 0 -1.57"/>
   </joint>
   </xacro:macro>

Commit message: Integrated new gripper (#50)
* Integrate CRACKLE_CLAW firmware and update claw degree publisher

- Added CRACKLE_CLAW submodule for claw control
- Implemented claw control logic in claw_degree_publisher
- Enhanced URDF with new gripper mesh and joint definitions
- Updated package dependencies for ROS integration

* Update CRACKLE_CLAW submodule to latest commit

* Added new gripper and edited description

* Fixed gripper and pick up pipeline issues

File: crackle_description/urdf/crackle_gripper.urdf.xacro (robot description, xacro)
@@ -5,51 +5,83 @@
   <xacro:property name="pkg_path" value="package://crackle_description/meshes"/>
   <xacro:property name="mesh_scale" value="1 1 1"/>
+  <!-- The lateral_rack_pinion_gripper mesh is authored in millimetres; scale to metres. -->
+  <xacro:property name="mm_scale" value="0.001 0.001 0.001"/>
   <xacro:property name="arm_last_link" value="${arm_link}"/>
+  <!-- Placement of the gripper mesh within the gripper_base link.
+       In the raw mesh the rack/pinion mechanism sits at one end (mesh Z=-196mm)
+       and the two fingers at the other (mesh Z=+38mm), with the lateral rack
+       running along mesh X. This transform mounts the mechanism end on the
+       flange (link origin) and points the fingers out along +Z (the arm's
+       approach direction), with the rack opening along Y. The 90° yaw turns
+       the rack from mesh X onto Y. -->
+  <xacro:property name="gripper_mesh_xyz" value="-0.002 0.020 0.196"/>
+  <xacro:property name="gripper_mesh_rpy" value="0 0 1.5708"/>
+  <!-- Lateral rack (jaw) travel, in metres, from fully open (0) to fully closed. -->
+  <xacro:property name="rack_travel" value="0.04"/>
+  <!-- Where the jaws sit relative to the base origin: near the finger tips
+       (+Z) and offset laterally along Y. -->
+  <xacro:property name="jaw_z" value="0.19"/>
+  <xacro:property name="jaw_open_y" value="0.05"/>
   <!-- =========================
        Macro: Gripper Base Link
        ========================= -->
-  <xacro:macro name="gripper_base_macro" params="link_name base_mesh:='ClawBase.stl'">
+  <xacro:macro name="gripper_base_macro" params="link_name base_mesh:='lateral_rack_pinion_gripper.stl'">
     <link name="${link_name}">
       <visual>
-        <origin xyz="0 0 0" rpy="0 0 1.80"/>
+        <origin xyz="${gripper_mesh_xyz}" rpy="${gripper_mesh_rpy}"/>
         <geometry>
-          <mesh filename="${pkg_path}/${base_mesh}" scale="${mesh_scale}"/>
+          <mesh filename="${pkg_path}/${base_mesh}" scale="${mm_scale}"/>
         </geometry>
+        <material name="gripper_blue">
+          <color rgba="0.0 0.0 0.5 1"/>
+        </material>
       </visual>
-      <color rgba="0.0 0.0 0.5 1"/>
     </link>
-<!--
-    <link name="spur_gear_left">
+    <!-- ===== Left rack (jaw) ===== -->
+    <link name="left_rack">
       <visual>
-        <origin xyz="0 0 0" rpy="0 0 1.80"/>
+        <origin xyz="0 0 0" rpy="0 0 0"/>
         <geometry>
-          <mesh filename="${pkg_path}/SpurGear.stl" scale="${mesh_scale}"/>
+          <box size="0.02 0.01 0.04"/>
         </geometry>
+        <material name="rack_grey">
+          <color rgba="0.3 0.3 0.3 1"/>
+        </material>
       </visual>
-      <color rgba="0.0 0.0 0.5 1"/>
     </link>
-  <link name="spur_gear_right">
+    <!-- ===== Right rack (jaw) ===== -->
+    <link name="right_rack">
       <visual>
-        <origin xyz="0 0 0" rpy="0 0 1.80"/>
+        <origin xyz="0 0 0" rpy="0 0 0"/>
         <geometry>
-          <mesh filename="${pkg_path}/SpurGear.stl" scale="${mesh_scale}"/>
+          <box size="0.02 0.01 0.04"/>
         </geometry>
+        <material name="rack_grey">
+          <color rgba="0.3 0.3 0.3 1"/>
+        </material>
       </visual>
-      <color rgba="0.0 0.0 0.5 1"/>
-  </link>
-    <joint name="spur_gear_left_joint" type="revolute">
+    </link>
+    <!-- Rack (jaw) joints, pinned FIXED at the open position for now.
+         They were prismatic (rack opens along Y, driven symmetrically by the
+         two pinion servos), but a movable joint has no transform until its
+         position is published on /joint_states — which only happens when the
+         claw node is running and the ESP32 is streaming. That broke TF
+         (no transform to left_rack) and MoveIt's current-state monitor
+         (incomplete state -> planning failures) whenever the gripper wasn't
+         actively driven. Fixed joints always resolve and add no DOF to MoveIt.
+         To re-enable articulation: set type="prismatic", restore the <axis>
+         (0 -1 0 / 0 1 0) and <limit lower="0.0" upper="${rack_travel}" ...>,
+         and make claw_degree_publisher publish these joints on /joint_states
+         continuously (see publish_joint_states param). -->
+    <joint name="left_rack_joint" type="fixed">
       <parent link="${link_name}"/>
-      <child link="spur_gear_left"/>
-      <origin xyz="0.0 0.02 0.03" rpy="3.14 1.57 0.3"/>
-      <axis xyz="0 0 1"/>
-      <limit lower="-3.14159" upper="3.14159" effort="5.0" velocity="5.0"/>
+      <child link="left_rack"/>
+      <origin xyz="0 ${jaw_open_y} ${jaw_z}" rpy="0 0 0"/>
     </joint>
-    <joint name="spur_gear_right_joint" type="revolute">
+    <joint name="right_rack_joint" type="fixed">
       <parent link="${link_name}"/>
-      <child link="spur_gear_right"/>
-      <origin xyz="0.0 -0.02 0.03" rpy="0 1.57 0.3"/>
-      <axis xyz="0 0 1"/>
-      <limit lower="-3.14159" upper="3.14159" effort="5.0" velocity="5.0"/>
-    </joint>  -->
+      <child link="right_rack"/>
+      <origin xyz="0 ${-jaw_open_y} ${jaw_z}" rpy="0 0 0"/>
+    </joint>
   </xacro:macro>
   <!-- =========================
@@ -58,9 +90,12 @@
   <!-- 1) Base link -->
   <xacro:gripper_base_macro link_name="gripper_base"/>
-  <!-- 2) Fixed joint to arm -->
+  <!-- 2) Fixed joint to arm. The mesh transform above already puts the mount
+       face at the gripper_base origin with the fingers along +Z, so the
+       gripper mounts flush on the flange. Adjust the yaw here to clock the
+       gripper about the tool axis if the jaw-opening direction needs rotating. -->
   <joint name="gripper_base_joint" type="fixed">
     <parent link="${arm_last_link}"/>
     <child link="gripper_base"/>
-    <origin xyz="0 0 0.025" rpy="0.0 0 -0.78"/> <!-- 0.78 -->
+    <origin xyz="0.0 0.0 0.0" rpy="0 0 0"/>
   </joint>
   <link name="camera_depth_optical_frame">
@@ -71,5 +106,5 @@
       </geometry>
       <material name="blue">
-        <color rgba="0.0 0.0 0.5 1"/>
+        <color rgba="0.5 0.0 0.0 1"/>
       </material>
     </visual>
@@ -85,5 +120,5 @@
     <parent link="gripper_base"/>
     <child link="camera_depth_optical_frame"/>
-    <origin xyz="-0.08 0 0.03" rpy="0 0 -1.57"/>
+    <origin xyz="0.02 0.02 0.05" rpy="0.04 0 -1.57"/>
   </joint>
   </xacro:macro>

Commit message: pickup pipeline improved consistence

File: crackle_description/urdf/crackle_gripper.urdf.xacro (robot description, xacro)
@@ -37,4 +37,15 @@
         </material>
       </visual>
+      <!-- Collision geometry so MoveIt actually sees the gripper body and stops
+           plans that would drive it through the table (or other obstacles). Uses
+           the same STL + transform as the visual, so the collision model matches
+           exactly what you see, INCLUDING the open gap between the fingers (so a
+           target object can still fit between them). -->
+      <collision>
+        <origin xyz="${gripper_mesh_xyz}" rpy="${gripper_mesh_rpy}"/>
+        <geometry>
+          <mesh filename="${pkg_path}/${base_mesh}" scale="${mm_scale}"/>
+        </geometry>
+      </collision>
     </link>
     <!-- ===== Left rack (jaw) ===== -->
@@ -49,4 +60,10 @@
         </material>
       </visual>
+      <collision>
+        <origin xyz="0 0 0" rpy="0 0 0"/>
+        <geometry>
+          <box size="0.02 0.01 0.04"/>
+        </geometry>
+      </collision>
     </link>
     <!-- ===== Right rack (jaw) ===== -->
@@ -61,4 +78,10 @@
         </material>
       </visual>
+      <collision>
+        <origin xyz="0 0 0" rpy="0 0 0"/>
+        <geometry>
+          <box size="0.02 0.01 0.04"/>
+        </geometry>
+      </collision>
     </link>
     <!-- Rack (jaw) joints, pinned FIXED at the open position for now.
@@ -97,5 +120,5 @@
     <parent link="${arm_last_link}"/>
     <child link="gripper_base"/>
-    <origin xyz="0.0 0.0 0.0" rpy="0 0 0"/>
+    <origin xyz="0.015 0.001 0.0" rpy="0 0 0"/>
   </joint>
   <link name="camera_depth_optical_frame">
@@ -117,8 +140,9 @@
     </inertial>
   </link>
+<!--"0.02 0.02 0.05" -->
   <joint name="camera_depth_optical_frame_joint" type="fixed">
     <parent link="gripper_base"/>
     <child link="camera_depth_optical_frame"/>
-    <origin xyz="0.02 0.02 0.05" rpy="0.04 0 -1.57"/>
+    <origin xyz="0.05 -0.005 0.057" rpy="0.04 0 -1.57"/>
   </joint>
   </xacro:macro>

File: xarm_ros2/xarm_moveit_config/srdf/_lite6_macro.srdf.xacro (robot description, xacro)
@@ -95,4 +95,23 @@
     <disable_collisions link1="${prefix}link5" link2="${prefix}link_eef" reason="Never" />
     <disable_collisions link1="${prefix}link6" link2="${prefix}link_eef" reason="Adjacent" />
+    <!-- ===== Crackle custom gripper (crackle_description/crackle_gripper.urdf.xacro) =====
+         The gripper links (gripper_base, left_rack, right_rack) now carry collision
+         geometry so MoveIt catches gripper-vs-table/obstacle collisions. Disable the
+         self-collisions between the gripper and the arm links it is mounted on, and
+         among the gripper's own links, or planning would fail on spurious contacts.
+         The gripper links are unprefixed (single-arm crackle setup). -->
+    <disable_collisions link1="${prefix}link6" link2="gripper_base" reason="Adjacent" />
+    <disable_collisions link1="${prefix}link_eef" link2="gripper_base" reason="Adjacent" />
+    <disable_collisions link1="${prefix}link5" link2="gripper_base" reason="Never" />
+    <disable_collisions link1="${prefix}link4" link2="gripper_base" reason="Never" />
+    <disable_collisions link1="${prefix}link6" link2="left_rack" reason="Never" />
+    <disable_collisions link1="${prefix}link6" link2="right_rack" reason="Never" />
+    <disable_collisions link1="${prefix}link_eef" link2="left_rack" reason="Never" />
+    <disable_collisions link1="${prefix}link_eef" link2="right_rack" reason="Never" />
+    <disable_collisions link1="${prefix}link5" link2="left_rack" reason="Never" />
+    <disable_collisions link1="${prefix}link5" link2="right_rack" reason="Never" />
+    <disable_collisions link1="gripper_base" link2="left_rack" reason="Adjacent" />
+    <disable_collisions link1="gripper_base" link2="right_rack" reason="Adjacent" />
+    <disable_collisions link1="left_rack" link2="right_rack" reason="Never" />
   </xacro:macro>
 </robot>
