Commit message: Improved pickup

File: crackle_description/urdf/crackle_gripper.urdf.xacro (robot description, xacro)
@@ -49,5 +49,9 @@
       </collision>
     </link>
-    <!-- ===== Left rack (jaw) ===== -->
+    <!-- ===== Left rack (jaw) =====
+         Visual only, NO collision: the racks are moving (prismatic) jaws that
+         close around the grasped object, so leaving them collidable just trips
+         false object/table collisions during grasp and lift. The gripper_base
+         mesh already provides the gripper body's collision geometry. -->
     <link name="left_rack">
       <visual>
@@ -60,12 +64,6 @@
         </material>
       </visual>
-      <collision>
-        <origin xyz="0 0 0" rpy="0 0 0"/>
-        <geometry>
-          <box size="0.02 0.01 0.04"/>
-        </geometry>
-      </collision>
     </link>
-    <!-- ===== Right rack (jaw) ===== -->
+    <!-- ===== Right rack (jaw) ===== visual only, NO collision (see left_rack). -->
     <link name="right_rack">
       <visual>
@@ -78,32 +76,26 @@
         </material>
       </visual>
-      <collision>
-        <origin xyz="0 0 0" rpy="0 0 0"/>
-        <geometry>
-          <box size="0.02 0.01 0.04"/>
-        </geometry>
-      </collision>
     </link>
-    <!-- Rack (jaw) joints, pinned FIXED at the open position for now.
-         They were prismatic (rack opens along Y, driven symmetrically by the
-         two pinion servos), but a movable joint has no transform until its
-         position is published on /joint_states — which only happens when the
-         claw node is running and the ESP32 is streaming. That broke TF
-         (no transform to left_rack) and MoveIt's current-state monitor
-         (incomplete state -> planning failures) whenever the gripper wasn't
-         actively driven. Fixed joints always resolve and add no DOF to MoveIt.
-         To re-enable articulation: set type="prismatic", restore the <axis>
-         (0 -1 0 / 0 1 0) and <limit lower="0.0" upper="${rack_travel}" ...>,
-         and make claw_degree_publisher publish these joints on /joint_states
-         continuously (see publish_joint_states param). -->
-    <joint name="left_rack_joint" type="fixed">
+    <!-- Rack (jaw) joints: PRISMATIC, driven symmetrically by the two pinion
+         servos. Position 0 = fully open, ${rack_travel} = fully closed; both
+         racks share the same (positive) value and close inward along ∓Y.
+         A movable joint has no TF until its position is published on
+         /joint_states, so claw_degree_publisher MUST publish these joints
+         continuously (publish_joint_states=true, defaulting to 0.0/open even
+         before the ESP32 streams). Without that, TF (world->left_rack) and
+         MoveIt's current-state monitor go incomplete and planning fails. -->
+    <joint name="left_rack_joint" type="prismatic">
       <parent link="${link_name}"/>
       <child link="left_rack"/>
       <origin xyz="0 ${jaw_open_y} ${jaw_z}" rpy="0 0 0"/>
+      <axis xyz="0 -1 0"/>
+      <limit lower="0.0" upper="${rack_travel}" effort="10.0" velocity="0.1"/>
     </joint>
-    <joint name="right_rack_joint" type="fixed">
+    <joint name="right_rack_joint" type="prismatic">
       <parent link="${link_name}"/>
       <child link="right_rack"/>
       <origin xyz="0 ${-jaw_open_y} ${jaw_z}" rpy="0 0 0"/>
+      <axis xyz="0 1 0"/>
+      <limit lower="0.0" upper="${rack_travel}" effort="10.0" velocity="0.1"/>
     </joint>
   </xacro:macro>

File: xarm_ros2/xarm_moveit_config/srdf/_lite6_macro.srdf.xacro (robot description, xacro)
@@ -43,4 +43,12 @@
       <joint name="${prefix}joint6" value="0" />
     </group_state>
+    <!-- crackle lateral rack-and-pinion gripper (always attached in the URDF).
+         The two rack jaws are PRISMATIC joints driven by the claw firmware, not
+         by motion planning, so mark them passive. Their positions are supplied
+         on /joint_states by claw_degree_publisher. Names are unprefixed because
+         the three_claw_gripper macro defines them without a prefix. The
+         gripper-link disable_collisions live in the block further below. -->
+    <passive_joint name="left_rack_joint" />
+    <passive_joint name="right_rack_joint" />
     <!-- gripper -->
     <xacro:if value="${add_gripper}">

Commit message: Tanay24/scanning (#53)
* pickup pipeline improved consistence

* Improved pickup

* Fixed pickup pipeline and added API functions

File: crackle_description/urdf/crackle_gripper.urdf.xacro (robot description, xacro)
@@ -37,6 +37,21 @@
         </material>
       </visual>
+      <!-- Collision geometry so MoveIt actually sees the gripper body and stops
+           plans that would drive it through the table (or other obstacles). Uses
+           the same STL + transform as the visual, so the collision model matches
+           exactly what you see, INCLUDING the open gap between the fingers (so a
+           target object can still fit between them). -->
+      <collision>
+        <origin xyz="${gripper_mesh_xyz}" rpy="${gripper_mesh_rpy}"/>
+        <geometry>
+          <mesh filename="${pkg_path}/${base_mesh}" scale="${mm_scale}"/>
+        </geometry>
+      </collision>
     </link>
-    <!-- ===== Left rack (jaw) ===== -->
+    <!-- ===== Left rack (jaw) =====
+         Visual only, NO collision: the racks are moving (prismatic) jaws that
+         close around the grasped object, so leaving them collidable just trips
+         false object/table collisions during grasp and lift. The gripper_base
+         mesh already provides the gripper body's collision geometry. -->
     <link name="left_rack">
       <visual>
@@ -50,5 +65,5 @@
       </visual>
     </link>
-    <!-- ===== Right rack (jaw) ===== -->
+    <!-- ===== Right rack (jaw) ===== visual only, NO collision (see left_rack). -->
     <link name="right_rack">
       <visual>
@@ -62,25 +77,25 @@
       </visual>
     </link>
-    <!-- Rack (jaw) joints, pinned FIXED at the open position for now.
-         They were prismatic (rack opens along Y, driven symmetrically by the
-         two pinion servos), but a movable joint has no transform until its
-         position is published on /joint_states — which only happens when the
-         claw node is running and the ESP32 is streaming. That broke TF
-         (no transform to left_rack) and MoveIt's current-state monitor
-         (incomplete state -> planning failures) whenever the gripper wasn't
-         actively driven. Fixed joints always resolve and add no DOF to MoveIt.
-         To re-enable articulation: set type="prismatic", restore the <axis>
-         (0 -1 0 / 0 1 0) and <limit lower="0.0" upper="${rack_travel}" ...>,
-         and make claw_degree_publisher publish these joints on /joint_states
-         continuously (see publish_joint_states param). -->
-    <joint name="left_rack_joint" type="fixed">
+    <!-- Rack (jaw) joints: PRISMATIC, driven symmetrically by the two pinion
+         servos. Position 0 = fully open, ${rack_travel} = fully closed; both
+         racks share the same (positive) value and close inward along ∓Y.
+         A movable joint has no TF until its position is published on
+         /joint_states, so claw_degree_publisher MUST publish these joints
+         continuously (publish_joint_states=true, defaulting to 0.0/open even
+         before the ESP32 streams). Without that, TF (world->left_rack) and
+         MoveIt's current-state monitor go incomplete and planning fails. -->
+    <joint name="left_rack_joint" type="prismatic">
       <parent link="${link_name}"/>
       <child link="left_rack"/>
       <origin xyz="0 ${jaw_open_y} ${jaw_z}" rpy="0 0 0"/>
+      <axis xyz="0 -1 0"/>
+      <limit lower="0.0" upper="${rack_travel}" effort="10.0" velocity="0.1"/>
     </joint>
-    <joint name="right_rack_joint" type="fixed">
+    <joint name="right_rack_joint" type="prismatic">
       <parent link="${link_name}"/>
       <child link="right_rack"/>
       <origin xyz="0 ${-jaw_open_y} ${jaw_z}" rpy="0 0 0"/>
+      <axis xyz="0 1 0"/>
+      <limit lower="0.0" upper="${rack_travel}" effort="10.0" velocity="0.1"/>
     </joint>
   </xacro:macro>
@@ -97,5 +112,5 @@
     <parent link="${arm_last_link}"/>
     <child link="gripper_base"/>
-    <origin xyz="0.0 0.0 0.0" rpy="0 0 0"/>
+    <origin xyz="0.015 0.001 0.0" rpy="0 0 0"/>
   </joint>
   <link name="camera_depth_optical_frame">
@@ -117,8 +132,9 @@
     </inertial>
   </link>
+<!--"0.02 0.02 0.05" -->
   <joint name="camera_depth_optical_frame_joint" type="fixed">
     <parent link="gripper_base"/>
     <child link="camera_depth_optical_frame"/>
-    <origin xyz="0.02 0.02 0.05" rpy="0.04 0 -1.57"/>
+    <origin xyz="0.05 -0.005 0.057" rpy="0.04 0 -1.57"/>
   </joint>
   </xacro:macro>

File: xarm_ros2/xarm_moveit_config/srdf/_lite6_macro.srdf.xacro (robot description, xacro)
@@ -43,4 +43,12 @@
       <joint name="${prefix}joint6" value="0" />
     </group_state>
+    <!-- crackle lateral rack-and-pinion gripper (always attached in the URDF).
+         The two rack jaws are PRISMATIC joints driven by the claw firmware, not
+         by motion planning, so mark them passive. Their positions are supplied
+         on /joint_states by claw_degree_publisher. Names are unprefixed because
+         the three_claw_gripper macro defines them without a prefix. The
+         gripper-link disable_collisions live in the block further below. -->
+    <passive_joint name="left_rack_joint" />
+    <passive_joint name="right_rack_joint" />
     <!-- gripper -->
     <xacro:if value="${add_gripper}">
@@ -95,4 +103,23 @@
     <disable_collisions link1="${prefix}link5" link2="${prefix}link_eef" reason="Never" />
     <disable_collisions link1="${prefix}link6" link2="${prefix}link_eef" reason="Adjacent" />
+    <!-- ===== Crackle custom gripper (crackle_description/crackle_gripper.urdf.xacro) =====
+         The gripper links (gripper_base, left_rack, right_rack) now carry collision
+         geometry so MoveIt catches gripper-vs-table/obstacle collisions. Disable the
+         self-collisions between the gripper and the arm links it is mounted on, and
+         among the gripper's own links, or planning would fail on spurious contacts.
+         The gripper links are unprefixed (single-arm crackle setup). -->
+    <disable_collisions link1="${prefix}link6" link2="gripper_base" reason="Adjacent" />
+    <disable_collisions link1="${prefix}link_eef" link2="gripper_base" reason="Adjacent" />
+    <disable_collisions link1="${prefix}link5" link2="gripper_base" reason="Never" />
+    <disable_collisions link1="${prefix}link4" link2="gripper_base" reason="Never" />
+    <disable_collisions link1="${prefix}link6" link2="left_rack" reason="Never" />
+    <disable_collisions link1="${prefix}link6" link2="right_rack" reason="Never" />
+    <disable_collisions link1="${prefix}link_eef" link2="left_rack" reason="Never" />
+    <disable_collisions link1="${prefix}link_eef" link2="right_rack" reason="Never" />
+    <disable_collisions link1="${prefix}link5" link2="left_rack" reason="Never" />
+    <disable_collisions link1="${prefix}link5" link2="right_rack" reason="Never" />
+    <disable_collisions link1="gripper_base" link2="left_rack" reason="Adjacent" />
+    <disable_collisions link1="gripper_base" link2="right_rack" reason="Adjacent" />
+    <disable_collisions link1="left_rack" link2="right_rack" reason="Never" />
   </xacro:macro>
 </robot>

Commit message: on the day fixes

File: crackle_description/urdf/crackle_gripper.urdf.xacro (robot description, xacro)
@@ -136,5 +136,6 @@
     <parent link="gripper_base"/>
     <child link="camera_depth_optical_frame"/>
-    <origin xyz="0.05 -0.005 0.057" rpy="0.04 0 -1.57"/>
+    <!-- was: <origin xyz="0.05 -0.005 0.057" rpy="0.04 0 -1.57"/> -->
+    <origin xyz="0.03810 0.03504 -0.02364" rpy="0.05900 -0.00253 -1.60644"/>
   </joint>
   </xacro:macro>

Commit message: more last day fixes

File: crackle_description/urdf/crackle_gripper.urdf.xacro (robot description, xacro)
@@ -136,6 +136,6 @@
     <parent link="gripper_base"/>
     <child link="camera_depth_optical_frame"/>
-    <!-- was: <origin xyz="0.05 -0.005 0.057" rpy="0.04 0 -1.57"/> -->
-    <origin xyz="0.03810 0.03504 -0.02364" rpy="0.05900 -0.00253 -1.60644"/>
+     <origin xyz="0.05 -0.005 0.057" rpy=".2 -.08 -1.57"/>
+    <!-- <origin xyz="0.03810 0.03504 -0.02364" rpy="0.05900 -0.00253 -1.60644"/> -->
   </joint>
   </xacro:macro>
